File: KiCad/Nuttali/file601B1424.sch (KiCad schematic (older format))
At the start: 17 parts

Commit message: Small changes on PMW
Parts:
- C? (x3): value C_Small -> 10uF
- C? (x3): value C_Small -> 100nF
- C?: value C_Small -> 100uF
- C?: value C_Small -> 4.7μF/10V
- R?: value R_Small -> 13
- R?: value R_Small -> 10k
- U?: symbol new_components:PMW3389 -> Nuttali-rescue:PMW3389-new_components
Other:
- moved on the sheet: C?, R?
