File: KiCad/Nuttali/file601B1424.sch (KiCad schematic (older format))
At the start: 17 parts

Commit message: Footprint
Parts:
- C14, C15, C16, C17, C18, C19, C20, C21: renamed from C?; footprint (none) -> Capacitor_SMD:C_0805_2012Metric_Pad1.18x1.45mm_HandSolder
- R2, R3: renamed from R?; footprint (none) -> Resistor_SMD:R_0805_2012Metric_Pad1.20x1.40mm_HandSolder
- TP1, TP2, TP3, TP4, TP5, TP6: renamed from TP?; footprint (none) -> TestPoint:TestPoint_2Pads_Pitch2.54mm_Drill0.8mm
- gave numbers to parts that had none: 1
Changed lines of the file:
@@
 $EndDescr
 $Comp
-L Nuttali-rescue:PMW3389-new_components U?
+L Nuttali-rescue:PMW3389-new_components U2
 U 1 1 601B49B3
 P 4700 2700
-F 0 "U?" H 4650 3265 50  0000 C CNN
+F 0 "U2" H 4650 3265 50  0000 C CNN
 F 1 "PMW3389" H 4650 3174 50  0000 C CNN
 F 2 "" H 4700 2150 50  0001 C CNN
@@
 $EndComp
 $Comp
-L power:+3.3V #PWR?
+L power:+3.3V #PWR0116
 U 1 1 601B6020
 P 2250 3500
-F 0 "#PWR?" H 2250 3350 50  0001 C CNN
+F 0 "#PWR0116" H 2250 3350 50  0001 C CNN
 F 1 "+3.3V" H 2265 3673 50  0000 C CNN
 F 2 "" H 2250 3500 50  0001 C CNN
@@
 $EndComp
 $Comp
-L Device:C_Small C?
+L Device:C_Small C16
 U 1 1 601B7149
 P 2500 3600
-F 0 "C?" H 2592 3646 50  0000 L CNN
+F 0 "C16" H 2592 3646 50  0000 L CNN
 F 1 "10uF" H 2592 3555 50  0000 L CNN
-F 2 "" H 2500 3600 50  0001 C CNN
+F 2 "Capacitor_SMD:C_0805_2012Metric_Pad1.18x1.45mm_HandSolder" H 2500 3600 50  0001 C CNN
 F 3 "~" H 2500 3600 50  0001 C CNN
 	1    2500 3600
@@
 $EndComp
 $Comp
-L Device:C_Small C?
+L Device:C_Small C19
 U 1 1 601B779D
 P 3000 3600
-F 0 "C?" H 3092 3646 50  0000 L CNN
+F 0 "C19" H 3092 3646 50  0000 L CNN
 F 1 "100nF" H 3092 3555 50  0000 L CNN
-F 2 "" H 3000 3600 50  0001 C CNN
+F 2 "Capacitor_SMD:C_0805_2012Metric_Pad1.18x1.45mm_HandSolder" H 3000 3600 50  0001 C CNN
 F 3 "~" H 3000 3600 50  0001 C CNN
 	1    3000 3600
@@
 $EndComp
 $Comp
-L power:GND #PWR?
+L power:GND #PWR0117
 U 1 1 601B7EF0
 P 2750 3800
-F 0 "#PWR?" H 2750 3550 50  0001 C CNN
+F 0 "#PWR0117" H 2750 3550 50  0001 C CNN
 F 1 "GND" H 2755 3627 50  0000 C CNN
 F 2 "" H 2750 3800 50  0001 C CNN
@@
 P 2250 2800
 AR Path="/601BB0BC" Ref="#PWR?"  Part="1"
-AR Path="/601B1425/601BB0BC" Ref="#PWR?"  Part="1"
-F 0 "#PWR?" H 2250 2650 50  0001 C CNN
+AR Path="/601B1425/601BB0BC" Ref="#PWR0118"  Part="1"
+F 0 "#PWR0118" H 2250 2650 50  0001 C CNN
 F 1 "+1.9V" H 2265 2973 50  0000 C CNN
 F 2 "" H 2250 2800 50  0001 C CNN
@@
 $EndComp
 $Comp
-L Device:C_Small C?
+L Device:C_Small C15
 U 1 1 601BBB39
 P 2500 2900
-F 0 "C?" H 2592 2946 50  0000 L CNN
+F 0 "C15" H 2592 2946 50  0000 L CNN
 F 1 "100uF" H 2592 2855 50  0000 L CNN
-F 2 "" H 2500 2900 50  0001 C CNN
+F 2 "Capacitor_SMD:C_0805_2012Metric_Pad1.18x1.45mm_HandSolder" H 2500 2900 50  0001 C CNN
 F 3 "~" H 2500 2900 50  0001 C CNN
 	1    2500 2900
@@
 $EndComp
 $Comp
-L Device:C_Small C?
+L Device:C_Small C18
 U 1 1 601BC32D
 P 3000 2900
-F 0 "C?" H 3092 2946 50  0000 L CNN
+F 0 "C18" H 3092 2946 50  0000 L CNN
 F 1 "10uF" H 3092 2855 50  0000 L CNN
-F 2 "" H 3000 2900 50  0001 C CNN
+F 2 "Capacitor_SMD:C_0805_2012Metric_Pad1.18x1.45mm_HandSolder" H 3000 2900 50  0001 C CNN
 F 3 "~" H 3000 2900 50  0001 C CNN
 	1    3000 2900
@@
 $EndComp
 $Comp
-L power:GND #PWR?
+L power:GND #PWR0119
 U 1 1 601BCBD9
 P 2750 3100
-F 0 "#PWR?" H 2750 2850 50  0001 C CNN
+F 0 "#PWR0119" H 2750 2850 50  0001 C CNN
 F 1 "GND" H 2755 2927 50  0000 C CNN
 F 2 "" H 2750 3100 50  0001 C CNN
@@
 Connection ~ 3000 2800
 $Comp
-L Device:C_Small C?
+L Device:C_Small C21
 U 1 1 601BE3E8
 P 7350 2550
-F 0 "C?" H 7442 2596 50  0000 L CNN
+F 0 "C21" H 7442 2596 50  0000 L CNN
 F 1 "100nF" H 7442 2505 50  0000 L CNN
-F 2 "" H 7350 2550 50  0001 C CNN
+F 2 "Capacitor_SMD:C_0805_2012Metric_Pad1.18x1.45mm_HandSolder" H 7350 2550 50  0001 C CNN
 F 3 "~" H 7350 2550 50  0001 C CNN
 	1    7350 2550
@@
 $EndComp
 $Comp
-L Device:C_Small C?
+L Device:C_Small C20
 U 1 1 601BEECD
 P 6850 2550
-F 0 "C?" H 6942 2596 50  0000 L CNN
+F 0 "C20" H 6942 2596 50  0000 L CNN
 F 1 "10uF" H 6942 2505 50  0000 L CNN
-F 2 "" H 6850 2550 50  0001 C CNN
+F 2 "Capacitor_SMD:C_0805_2012Metric_Pad1.18x1.45mm_HandSolder" H 6850 2550 50  0001 C CNN
 F 3 "~" H 6850 2550 50  0001 C CNN
 	1    6850 2550
@@
 $EndComp
 $Comp
-L power:GND #PWR?
+L power:GND #PWR0120
 U 1 1 601BFAD1
 P 7050 2750
-F 0 "#PWR?" H 7050 2500 50  0001 C CNN
+F 0 "#PWR0120" H 7050 2500 50  0001 C CNN
 F 1 "GND" H 7055 2577 50  0000 C CNN
 F 2 "" H 7050 2750 50  0001 C CNN
@@
 Connection ~ 7050 2650
 $Comp
-L Device:R_Small R?
+L Device:R_Small R3
 U 1 1 601C1642
 P 6500 2450
-F 0 "R?" V 6304 2450 50  0000 C CNN
+F 0 "R3" V 6304 2450 50  0000 C CNN
 F 1 "13" V 6395 2450 50  0000 C CNN
-F 2 "" H 6500 2450 50  0001 C CNN
+F 2 "Resistor_SMD:R_0805_2012Metric_Pad1.20x1.40mm_HandSolder" H 6500 2450 50  0001 C CNN
 F 3 "~" H 6500 2450 50  0001 C CNN
 	1    6500 2450
@@
 P 7550 2450
 AR Path="/601C32CC" Ref="#PWR?"  Part="1"
-AR Path="/601B1425/601C32CC" Ref="#PWR?"  Part="1"
-F 0 "#PWR?" H 7550 2300 50  0001 C CNN
+AR Path="/601B1425/601C32CC" Ref="#PWR0121"  Part="1"
+F 0 "#PWR0121" H 7550 2300 50  0001 C CNN
 F 1 "+1.9V" H 7565 2623 50  0000 C CNN
 F 2 "" H 7550 2450 50  0001 C CNN
@@
 	5050 2800 5400 2800
 $Comp
-L Device:C_Small C?
+L Device:C_Small C14
 U 1 1 601CD863
 P 2450 2050
-F 0 "C?" H 2542 2096 50  0000 L CNN
+F 0 "C14" H 2542 2096 50  0000 L CNN
 F 1 "100nF" H 2542 2005 50  0000 L CNN
-F 2 "" H 2450 2050 50  0001 C CNN
+F 2 "Capacitor_SMD:C_0805_2012Metric_Pad1.18x1.45mm_HandSolder" H 2450 2050 50  0001 C CNN
 F 3 "~" H 2450 2050 50  0001 C CNN
 	1    2450 2050
@@
 $EndComp
 $Comp
-L Device:C_Small C?
+L Device:C_Small C17
 U 1 1 601CE396
 P 2950 2050
-F 0 "C?" H 3042 2096 50  0000 L CNN
+F 0 "C17" H 3042 2096 50  0000 L CNN
 F 1 "4.7μF/10V" H 3042 2005 50  0000 L CNN
-F 2 "" H 2950 2050 50  0001 C CNN
+F 2 "Capacitor_SMD:C_0805_2012Metric_Pad1.18x1.45mm_HandSolder" H 2950 2050 50  0001 C CNN
 F 3 "~" H 2950 2050 50  0001 C CNN
 	1    2950 2050
@@
 $EndComp
 $Comp
-L power:GND #PWR?
+L power:GND #PWR0122
 U 1 1 601CF8BA
 P 2950 2300
-F 0 "#PWR?" H 2950 2050 50  0001 C CNN
+F 0 "#PWR0122" H 2950 2050 50  0001 C CNN
 F 1 "GND" H 2955 2127 50  0000 C CNN
 F 2 "" H 2950 2300 50  0001 C CNN
@@
 Connection ~ 2950 2150
 $Comp
-L power:GND #PWR?
+L power:GND #PWR0123
 U 1 1 601D9FB5
 P 4150 3250
-F 0 "#PWR?" H 4150 3000 50  0001 C CNN
+F 0 "#PWR0123" H 4150 3000 50  0001 C CNN
 F 1 "GND" H 4155 3077 50  0000 C CNN
 F 2 "" H 4150 3250 50  0001 C CNN
@@
 Connection ~ 5400 2800
 $Comp
-L Connector:TestPoint TP?
+L Connector:TestPoint TP1
 U 1 1 60204BFD
 P 4950 3850
-F 0 "TP?" H 5008 3968 50  0000 L CNN
+F 0 "TP1" H 5008 3968 50  0000 L CNN
 F 1 "TestPoint" H 5008 3877 50  0000 L CNN
-F 2 "" H 5150 3850 50  0001 C CNN
+F 2 "TestPoint:TestPoint_2Pads_Pitch2.54mm_Drill0.8mm" H 5150 3850 50  0001 C CNN
 F 3 "~" H 5150 3850 50  0001 C CNN
 	1    4950 3850
@@
 $EndComp
 $Comp
-L power:GND #PWR?
+L power:GND #PWR0124
 U 1 1 60205A5B
 P 4950 3850
-F 0 "#PWR?" H 4950 3600 50  0001 C CNN
+F 0 "#PWR0124" H 4950 3600 50  0001 C CNN
 F 1 "GND" H 4955 3677 50  0000 C CNN
 F 2 "" H 4950 3850 50  0001 C CNN
@@
 $EndComp
 $Comp
-L Connector:TestPoint TP?
+L Connector:TestPoint TP2
 U 1 1 6020633C
 P 5400 3850
-F 0 "TP?" H 5458 3968 50  0000 L CNN
+F 0 "TP2" H 5458 3968 50  0000 L CNN
 F 1 "TestPoint" H 5458 3877 50  0000 L CNN
-F 2 "" H 5600 3850 50  0001 C CNN
+F 2 "TestPoint:TestPoint_2Pads_Pitch2.54mm_Drill0.8mm" H 5600 3850 50  0001 C CNN
 F 3 "~" H 5600 3850 50  0001 C CNN
 	1    5400 3850
@@
 $EndComp
 $Comp
-L Connector:TestPoint TP?
+L Connector:TestPoint TP3
 U 1 1 602068E2
 P 5900 3850
-F 0 "TP?" H 5958 3968 50  0000 L CNN
+F 0 "TP3" H 5958 3968 50  0000 L CNN
 F 1 "TestPoint" H 5958 3877 50  0000 L CNN
-F 2 "" H 6100 3850 50  0001 C CNN
+F 2 "TestPoint:TestPoint_2Pads_Pitch2.54mm_Drill0.8mm" H 6100 3850 50  0001 C CNN
 F 3 "~" H 6100 3850 50  0001 C CNN
 	1    5900 3850
@@
 MOSI
 $Comp
-L Connector:TestPoint TP?
+L Connector:TestPoint TP4
 U 1 1 602082AE
 P 6350 3850
-F 0 "TP?" H 6408 3968 50  0000 L CNN
+F 0 "TP4" H 6408 3968 50  0000 L CNN
 F 1 "TestPoint" H 6408 3877 50  0000 L CNN
-F 2 "" H 6550 3850 50  0001 C CNN
+F 2 "TestPoint:TestPoint_2Pads_Pitch2.54mm_Drill0.8mm" H 6550 3850 50  0001 C CNN
 F 3 "~" H 6550 3850 50  0001 C CNN
 	1    6350 3850
@@
 $EndComp
 $Comp
-L Connector:TestPoint TP?
+L Connector:TestPoint TP5
 U 1 1 6020880C
 P 6800 3850
-F 0 "TP?" H 6858 3968 50  0000 L CNN
+F 0 "TP5" H 6858 3968 50  0000 L CNN
 F 1 "TestPoint" H 6858 3877 50  0000 L CNN
-F 2 "" H 7000 3850 50  0001 C CNN
+F 2 "TestPoint:TestPoint_2Pads_Pitch2.54mm_Drill0.8mm" H 7000 3850 50  0001 C CNN
 F 3 "~" H 7000 3850 50  0001 C CNN
 	1    6800 3850
@@
 NCS
 $Comp
-L Connector:TestPoint TP?
+L Connector:TestPoint TP6
 U 1 1 602091FD
 P 7250 3850
-F 0 "TP?" H 7308 3968 50  0000 L CNN
+F 0 "TP6" H 7308 3968 50  0000 L CNN
 F 1 "TestPoint" H 7308 3877 50  0000 L CNN
-F 2 "" H 7450 3850 50  0001 C CNN
+F 2 "TestPoint:TestPoint_2Pads_Pitch2.54mm_Drill0.8mm" H 7450 3850 50  0001 C CNN
 F 3 "~" H 7450 3850 50  0001 C CNN
 	1    7250 3850
@@
 	5400 1850 5400 2000
 $Comp
-L Device:R_Small R?
+L Device:R_Small R2
 U 1 1 601C973A
 P 5400 2100
-F 0 "R?" H 5341 2054 50  0000 R CNN
+F 0 "R2" H 5341 2054 50  0000 R CNN
 F 1 "10k" H 5341 2145 50  0000 R CNN
-F 2 "" H 5400 2100 50  0001 C CNN
+F 2 "Resistor_SMD:R_0805_2012Metric_Pad1.20x1.40mm_HandSolder" H 5400 2100 50  0001 C CNN
 F 3 "~" H 5400 2100 50  0001 C CNN
 	1    5400 2100
@@
 $EndComp
 $Comp
-L power:+3.3V #PWR?
+L power:+3.3V #PWR0125
 U 1 1 601C8D0A
 P 5400 1850
-F 0 "#PWR?" H 5400 1700 50  0001 C CNN
+F 0 "#PWR0125" H 5400 1700 50  0001 C CNN
 F 1 "+3.3V" H 5415 2023 50  0000 C CNN
 F 2 "" H 5400 1850 50  0001 C CNN
