File: KiCad/Nuttali/file601B1424.sch (KiCad schematic (older format))
At the start: 17 parts, among them U2 PMW3389

Commit message: all footprints fixed
Parts:
- TP1, TP2, TP3, TP4, TP5, TP6: footprint TestPoint:TestPoint_2Pads_Pitch2.54mm_Drill0.8mm -> TestPoint:TestPoint_Pad_1.0x1.0mm
Changed lines of the file:
@@
 F 0 "TP1" H 5008 3968 50  0000 L CNN
 F 1 "TestPoint" H 5008 3877 50  0000 L CNN
-F 2 "TestPoint:TestPoint_2Pads_Pitch2.54mm_Drill0.8mm" H 5150 3850 50  0001 C CNN
+F 2 "TestPoint:TestPoint_Pad_1.0x1.0mm" H 5150 3850 50  0001 C CNN
 F 3 "~" H 5150 3850 50  0001 C CNN
 	1    4950 3850
@@
 F 0 "TP2" H 5458 3968 50  0000 L CNN
 F 1 "TestPoint" H 5458 3877 50  0000 L CNN
-F 2 "TestPoint:TestPoint_2Pads_Pitch2.54mm_Drill0.8mm" H 5600 3850 50  0001 C CNN
+F 2 "TestPoint:TestPoint_Pad_1.0x1.0mm" H 5600 3850 50  0001 C CNN
 F 3 "~" H 5600 3850 50  0001 C CNN
 	1    5400 3850
@@
 F 0 "TP3" H 5958 3968 50  0000 L CNN
 F 1 "TestPoint" H 5958 3877 50  0000 L CNN
-F 2 "TestPoint:TestPoint_2Pads_Pitch2.54mm_Drill0.8mm" H 6100 3850 50  0001 C CNN
+F 2 "TestPoint:TestPoint_Pad_1.0x1.0mm" H 6100 3850 50  0001 C CNN
 F 3 "~" H 6100 3850 50  0001 C CNN
 	1    5900 3850
@@
 F 0 "TP4" H 6408 3968 50  0000 L CNN
 F 1 "TestPoint" H 6408 3877 50  0000 L CNN
-F 2 "TestPoint:TestPoint_2Pads_Pitch2.54mm_Drill0.8mm" H 6550 3850 50  0001 C CNN
+F 2 "TestPoint:TestPoint_Pad_1.0x1.0mm" H 6550 3850 50  0001 C CNN
 F 3 "~" H 6550 3850 50  0001 C CNN
 	1    6350 3850
@@
 F 0 "TP5" H 6858 3968 50  0000 L CNN
 F 1 "TestPoint" H 6858 3877 50  0000 L CNN
-F 2 "TestPoint:TestPoint_2Pads_Pitch2.54mm_Drill0.8mm" H 7000 3850 50  0001 C CNN
+F 2 "TestPoint:TestPoint_Pad_1.0x1.0mm" H 7000 3850 50  0001 C CNN
 F 3 "~" H 7000 3850 50  0001 C CNN
 	1    6800 3850
@@
 F 0 "TP6" H 7308 3968 50  0000 L CNN
 F 1 "TestPoint" H 7308 3877 50  0000 L CNN
-F 2 "TestPoint:TestPoint_2Pads_Pitch2.54mm_Drill0.8mm" H 7450 3850 50  0001 C CNN
+F 2 "TestPoint:TestPoint_Pad_1.0x1.0mm" H 7450 3850 50  0001 C CNN
 F 3 "~" H 7450 3850 50  0001 C CNN
 	1    7250 3850

Commit message: First draft of the pcb
Connections:
- net SCLK renamed SCK

Commit message: extended the pcb board with 2 mm to right
Parts:
- C14, C15, C16, C17, C18, C19, C20, C21: symbol Device:C_Small -> Nuttali-rescue:C_Small-Device
- R2, R3: symbol Device:R_Small -> Nuttali-rescue:R_Small-Device
- TP1, TP2, TP3, TP4, TP5, TP6: symbol Connector:TestPoint -> Nuttali-rescue:TestPoint-Connector
Changed lines of the file:
@@
 $EndDescr
 $Comp
-L power:+3.3V #PWR0125
+L Nuttali-rescue:+3.3V-power #PWR0125
 U 1 1 601C8D0A
 P 5400 1850
@@
 $EndComp
 $Comp
-L Device:R_Small R2
+L Nuttali-rescue:R_Small-Device R2
 U 1 1 601C973A
 P 5400 2100
@@
 	5400 2800 5400 2200
 $Comp
-L Connector:TestPoint TP6
+L Nuttali-rescue:TestPoint-Connector TP6
 U 1 1 602091FD
 P 7250 3850
@@
 SCK
 $Comp
-L Connector:TestPoint TP5
+L Nuttali-rescue:TestPoint-Connector TP5
 U 1 1 6020880C
 P 6800 3850
@@
 $EndComp
 $Comp
-L Connector:TestPoint TP4
+L Nuttali-rescue:TestPoint-Connector TP4
 U 1 1 602082AE
 P 6350 3850
@@
 MISO
 $Comp
-L Connector:TestPoint TP3
+L Nuttali-rescue:TestPoint-Connector TP3
 U 1 1 602068E2
 P 5900 3850
@@
 $EndComp
 $Comp
-L Connector:TestPoint TP2
+L Nuttali-rescue:TestPoint-Connector TP2
 U 1 1 6020633C
 P 5400 3850
@@
 $EndComp
 $Comp
-L power:GND #PWR0124
+L Nuttali-rescue:GND-power #PWR0124
 U 1 1 60205A5B
 P 4950 3850
@@
 $EndComp
 $Comp
-L Connector:TestPoint TP1
+L Nuttali-rescue:TestPoint-Connector TP1
 U 1 1 60204BFD
 P 4950 3850
@@
 	4250 3100 4150 3100
 $Comp
-L power:GND #PWR0123
+L Nuttali-rescue:GND-power #PWR0123
 U 1 1 601D9FB5
 P 4150 3250
@@
 	2950 1850 3200 1850
 $Comp
-L power:GND #PWR0122
+L Nuttali-rescue:GND-power #PWR0122
 U 1 1 601CF8BA
 P 2950 2300
@@
 Connection ~ 2950 2150
 $Comp
-L Device:C_Small C17
+L Nuttali-rescue:C_Small-Device C17
 U 1 1 601CE396
 P 2950 2050
@@
 $EndComp
 $Comp
-L Device:C_Small C14
+L Nuttali-rescue:C_Small-Device C14
 U 1 1 601CD863
 P 2450 2050
@@
 	6400 2450 6250 2450
 $Comp
-L Device:R_Small R3
+L Nuttali-rescue:R_Small-Device R3
 U 1 1 601C1642
 P 6500 2450
@@
 	7350 2650 7050 2650
 $Comp
-L power:GND #PWR0120
+L Nuttali-rescue:GND-power #PWR0120
 U 1 1 601BFAD1
 P 7050 2750
@@
 Connection ~ 6850 2450
 $Comp
-L Device:C_Small C20
+L Nuttali-rescue:C_Small-Device C20
 U 1 1 601BEECD
 P 6850 2550
@@
 Connection ~ 7350 2450
 $Comp
-L Device:C_Small C21
+L Nuttali-rescue:C_Small-Device C21
 U 1 1 601BE3E8
 P 7350 2550
@@
 	2500 3000 2750 3000
 $Comp
-L power:GND #PWR0119
+L Nuttali-rescue:GND-power #PWR0119
 U 1 1 601BCBD9
 P 2750 3100
@@
 Connection ~ 3000 2800
 $Comp
-L Device:C_Small C18
+L Nuttali-rescue:C_Small-Device C18
 U 1 1 601BC32D
 P 3000 2900
@@
 Connection ~ 2500 2800
 $Comp
-L Device:C_Small C15
+L Nuttali-rescue:C_Small-Device C15
 U 1 1 601BBB39
 P 2500 2900
@@
 	2500 3700 2750 3700
 $Comp
-L power:GND #PWR0117
+L Nuttali-rescue:GND-power #PWR0117
 U 1 1 601B7EF0
 P 2750 3800
@@
 	3000 3500 3350 3500
 $Comp
-L Device:C_Small C19
+L Nuttali-rescue:C_Small-Device C19
 U 1 1 601B779D
 P 3000 3600
@@
 Connection ~ 2500 3500
 $Comp
-L Device:C_Small C16
+L Nuttali-rescue:C_Small-Device C16
 U 1 1 601B7149
 P 2500 3600
@@
 $EndComp
 $Comp
-L power:+3.3V #PWR0116
+L Nuttali-rescue:+3.3V-power #PWR0116
 U 1 1 601B6020
 P 2250 3500

Commit message: Fixed almost all footprints and nearly the layout of the pcb
Parts:
- U2: footprint PMW:PMW3389 -> Nuttali:PMW3389DM-T3QU
Changed lines of the file:
@@
 F 0 "U2" H 4650 3265 50  0000 C CNN
 F 1 "PMW3389" H 4650 3174 50  0000 C CNN
-F 2 "PMW:PMW3389" H 4700 2150 50  0001 C CNN
+F 2 "Nuttali:PMW3389DM-T3QU" H 4700 2150 50  0001 C CNN
 F 3 "" H 4700 2150 50  0001 C CNN
 	1    4700 2700

Commit message: Finnished the pcb
Changed lines of the file:
@@
 	1    0    0    -1
 $EndComp
-Wire Wire Line
-	3000 3500 3350 3500
 $Comp
 L Nuttali-rescue:C_Small-Device C19
@@
 VDDPIX
 Connection ~ 2950 1850
-Text GLabel 3350 3500 2    50   Input ~ 0
-VDDIO_3.3V
 Connection ~ 3000 3500
 Text GLabel 5050 2500 2    50   Output ~ 0
@@
 Text GLabel 4250 2600 0    50   Output ~ 0
 VDDPIX
-Text GLabel 4250 2800 0    50   Output ~ 0
-VDDIO_3.3V
 Wire Wire Line
 	4250 2700 3400 2700
 Wire Wire Line
 	3400 2700 3400 2800
+Wire Wire Line
+	3650 3500 3650 2800
+Wire Wire Line
+	3650 2800 4250 2800
+Wire Wire Line
+	3000 3500 3650 3500
 $EndSCHEMATC
