File: KiCad/Nuttali/MCU.sch (KiCad schematic (older format))
At the start: 19 parts

Commit message: some footprints fixed
Parts:
- C1, C10, C11, C12, C13, C2, C3, C4, C5, C6, C7, C8, C9: renamed from C?; footprint (none) -> Capacitor_SMD:C_0805_2012Metric_Pad1.18x1.45mm_HandSolder; symbol Device:C -> Nuttali-rescue:C-Device
- J1: renamed from J?; symbol Connector:Conn_01x06_Male -> Nuttali-rescue:Conn_01x06_Male-Connector
- R1: renamed from R?; footprint (none) -> Resistor_SMD:R_0815_2038Metric_Pad1.20x4.05mm_HandSolder; symbol Device:R -> Nuttali-rescue:R-Device
- SW1, SW2: renamed from SW?; symbol Switch:SW_SPDT -> Nuttali-rescue:SW_SPDT-Switch
- U1: renamed from U?; symbol MCU_ST_STM32F4:STM32F411RETx -> Nuttali-rescue:STM32F411RETx-MCU_ST_STM32F4
- Y1: renamed from Y?; symbol Device:Crystal -> Nuttali-rescue:Crystal-Device
Other:
- moved on the sheet: SW1
