File: KiCad/Nuttali/MCU.sch (KiCad schematic (older format))
At the start: 19 parts, among them J1 SWD, SW1 SW_DPST_x2, SW2 RND 210-00662, U1 STM32F411RETx, Y1 16Mhz

Commit message: all footprints fixed
Parts:
- added D5, D6, D7: LED_RGB, LED_SMD:LED_RGB_5050-6, symbol Device:LED_RGB
- added R16, R17, R18, R19, R20, R21, R22, R23, R24: 220, Resistor_SMD:R_0805_2012Metric_Pad1.20x1.40mm_HandSolder, symbol Device:R_Small
- added TP7, TP8, TP9: TestPoint, TestPoint:TestPoint_Pad_1.0x1.0mm, symbol Connector:TestPoint
- Y1: footprint (none) -> nya:Crystal_SMD_0603-2Pin_6.0x3.5mm_HandSoldering
Connections:
- net D+: now also TP8.1
- net D-: now also TP7.1
- net GND: now also R16.1, R17.1, R18.1, R19.1, R20.1, R21.1, R22.1, R23.1, R24.1, TP9.1
- net R_LED: now reaches U1.15 (PA1)
- net R_LED: now also D5.4 (BA), D6.4 (BA), D7.4 (BA)
- net G_LED: now reaches U1.16 (PA2)
- net G_LED: now also D5.5 (GA), D6.5 (GA), D7.5 (GA)
- net B_LED: now reaches U1.17 (PA3)
- net B_LED: now also D5.6 (RA), D6.6 (RA), D7.6 (RA)
- new net: D7.1 (RK), R24.2
- new net: D7.2 (GK), R23.2
- new net: D7.3 (BK), R22.2
- new net: D6.1 (RK), R21.2
- new net: D6.2 (GK), R20.2
- new net: D6.3 (BK), R19.2
- new net: D5.1 (RK), R18.2
- new net: D5.2 (GK), R17.2
- new net: D5.3 (BK), R16.2
- no-connect marks 36 -> 33
Other:
- moved on the sheet: J1

Commit message: First draft of the pcb
Connections:
- net B_LED: now also D5.4 (BA), D6.4 (BA), D7.4 (BA); no longer D5.6 (RA), D6.6 (RA), D7.6 (RA)
- net R_LED: now also D5.6 (RA), D6.6 (RA), D7.6 (RA); no longer D5.4 (BA), D6.4 (BA), D7.4 (BA)
- net Turbo: now reaches U1.20 (PA4)
- net RightB: now reaches U1.21 (PA5)
- net WheelButton: now reaches U1.22 (PA6)
- net WheelB: now reaches U1.23 (PA7)
- net WheelA: now reaches U1.24 (PC4)
- net LeftB: now reaches U1.25 (PC5)
- net Turbo_LED: now reaches U1.26 (PB0)
- net SideFront: now reaches U1.35 (PB14)
- net SideBack: now reaches U1.36 (PB15)
- no-connect marks 33 -> 25
Other:
- moved on the sheet: TP9

Commit message: extended the pcb board with 2 mm to right
Parts:
- D5, D6, D7: symbol Device:LED_RGB -> Nuttali-rescue:LED_RGB-Device
- J1: symbol Connector:Conn_01x06_Male -> Nuttali-rescue:Conn_01x06_Male-Connector
- R1: symbol Device:R -> Nuttali-rescue:R-Device
- R16, R17, R18, R19, R20, R21, R22, R23, R24: symbol Device:R_Small -> Nuttali-rescue:R_Small-Device
- SW1: symbol Switch:SW_DPST_x2 -> Nuttali-rescue:SW_DPST_x2-Switch
- SW2: symbol Switch:SW_SPDT -> Nuttali-rescue:SW_SPDT-Switch
- TP7, TP8, TP9: symbol Connector:TestPoint -> Nuttali-rescue:TestPoint-Connector
- Y1: symbol Device:Crystal -> Nuttali-rescue:Crystal-Device
Changed lines of the file:
@@
 2*(Cload-Cstray)*2^(18-6)= \n24pF = 22pF
 $Comp
-L Device:Crystal Y1
+L Nuttali-rescue:Crystal-Device Y1
 U 1 1 602B614B
 P 4300 3950
@@
 	4650 2850 4750 2850
 $Comp
-L Connector:Conn_01x06_Male J1
+L Nuttali-rescue:Conn_01x06_Male-Connector J1
 U 1 1 602DCAE5
 P 8400 5950
@@
 $EndComp
 $Comp
-L Switch:SW_SPDT SW2
+L Nuttali-rescue:SW_SPDT-Switch SW2
 U 1 1 602EAC7D
 P 3200 1450
@@
 	3000 1550 3000 1700
 $Comp
-L Device:R R1
+L Nuttali-rescue:R-Device R1
 U 1 1 602EF78F
 P 3000 1850
@@
 	7950 5650 7950 5600
 $Comp
-L power:+3.3V #PWR0114
+L Nuttali-rescue:+3.3V-power #PWR0114
 U 1 1 601F634D
 P 7950 5600
@@
 $EndComp
 $Comp
-L power:GND #PWR0115
+L Nuttali-rescue:GND-power #PWR0115
 U 1 1 601F695B
 P 7450 5900
@@
 NoConn ~ 4750 4350
 $Comp
-L Switch:SW_DPST_x2 SW1
+L Nuttali-rescue:SW_DPST_x2-Switch SW1
 U 1 1 60245B0E
 P 3150 2850
@@
 	3350 2850 3350 2900
 $Comp
-L Connector:TestPoint TP9
+L Nuttali-rescue:TestPoint-Connector TP9
 U 1 1 60242CC3
 P 6650 5950
@@
 Connection ~ 5850 5950
 $Comp
-L Connector:TestPoint TP7
+L Nuttali-rescue:TestPoint-Connector TP7
 U 1 1 6024AE5A
 P 2750 5450
@@
 $EndComp
 $Comp
-L Connector:TestPoint TP8
+L Nuttali-rescue:TestPoint-Connector TP8
 U 1 1 6024B3CD
 P 3250 5450
@@
 $EndComp
 $Comp
-L Device:R_Small R24
+L Nuttali-rescue:R_Small-Device R24
 U 1 1 6032C1C8
 P 9100 4500
@@
 $EndComp
 $Comp
-L Device:R_Small R23
+L Nuttali-rescue:R_Small-Device R23
 U 1 1 6032C1C2
 P 9100 4300
@@
 $EndComp
 $Comp
-L Device:R_Small R22
+L Nuttali-rescue:R_Small-Device R22
 U 1 1 6032C1BC
 P 9100 4100
@@
 $EndComp
 $Comp
-L Device:R_Small R21
+L Nuttali-rescue:R_Small-Device R21
 U 1 1 60329EB6
 P 9100 3650
@@
 $EndComp
 $Comp
-L Device:R_Small R20
+L Nuttali-rescue:R_Small-Device R20
 U 1 1 60329EB0
 P 9100 3450
@@
 $EndComp
 $Comp
-L Device:R_Small R19
+L Nuttali-rescue:R_Small-Device R19
 U 1 1 60329EAA
 P 9100 3250
@@
 $EndComp
 $Comp
-L Device:R_Small R18
+L Nuttali-rescue:R_Small-Device R18
 U 1 1 60327306
 P 9100 2800
@@
 $EndComp
 $Comp
-L Device:R_Small R17
+L Nuttali-rescue:R_Small-Device R17
 U 1 1 60326D05
 P 9100 2600
@@
 $EndComp
 $Comp
-L Device:R_Small R16
+L Nuttali-rescue:R_Small-Device R16
 U 1 1 6032557E
 P 9100 2400
@@
 $EndComp
 $Comp
-L Device:LED_RGB D5
+L Nuttali-rescue:LED_RGB-Device D5
 U 1 1 60285E04
 P 8550 2600
@@
 $EndComp
 $Comp
-L Device:LED_RGB D6
+L Nuttali-rescue:LED_RGB-Device D6
 U 1 1 602851F0
 P 8550 3450
@@
 $EndComp
 $Comp
-L Device:LED_RGB D7
+L Nuttali-rescue:LED_RGB-Device D7
 U 1 1 6028314D
 P 8550 4300

Commit message: Finnished the pcb
Connections:
- net B_LED: now also U1.15 (PA1); no longer U1.17 (PA3)
- net R_LED: now also U1.17 (PA3); no longer U1.15 (PA1)
- net WheelA: now also U1.23 (PA7); no longer U1.24 (PC4)
- net WheelB: now also U1.24 (PC4); no longer U1.23 (PA7)
Changed lines of the file:
@@
 Text GLabel 4650 2850 0    50   Input ~ 0
 BOOT0
-Text GLabel 6150 2750 2    50   Input ~ 0
+Text GLabel 6150 2950 2    50   Input ~ 0
 R_LED
 Text GLabel 6150 2850 2    50   Input ~ 0
 G_LED
-Text GLabel 6150 2950 2    50   Input ~ 0
-B_LED
 Text GLabel 8350 2800 0    50   Output ~ 0
 R_LED
@@
 Text GLabel 6150 4350 2    50   Input ~ 0
 Turbo_LED
-Text GLabel 6150 3050 2    50   Output ~ 0
-Turbo
-Text GLabel 6150 3350 2    50   Input ~ 0
+Text GLabel 4750 4650 0    50   Input ~ 0
 WheelB
-Text GLabel 4750 4650 0    50   Input ~ 0
-WheelA
 Text GLabel 6150 3250 2    50   Output ~ 0
 WheelButton
@@
 Text GLabel 4750 4750 0    50   Output ~ 0
 LeftB
-Text GLabel 6150 3150 2    50   Output ~ 0
-RightB
 NoConn ~ 6150 3450
 NoConn ~ 6150 3550
@@
 Wire Wire Line
 	5850 5950 6650 5950
+Text GLabel 6150 3050 2    50   Output ~ 0
+Turbo
+Text GLabel 6150 2750 2    50   Input ~ 0
+B_LED
+Text GLabel 6150 3150 2    50   Output ~ 0
+RightB
+Text GLabel 6150 3350 2    50   Input ~ 0
+WheelA
 $EndSCHEMATC

Commit message: Finnished design.
Parts:
- removed D5, D6, D7: LED_RGB, LED_SMD:LED_RGB_5050-6, symbol Nuttali-rescue:LED_RGB-Device
- removed R19, R20, R21, R22, R23, R24: 220, Resistor_SMD:R_0805_2012Metric_Pad1.20x1.40mm_HandSolder, symbol Nuttali-rescue:R_Small-Device
- added J5: Conn_01x04_Male, Connector_PinSocket_2.54mm:PinSocket_1x04_P2.54mm_Vertical, symbol Connector:Conn_01x04_Male
Connections:
- net B_LED: now also R18.2
- net GND: now also J5.1 (Pin_1); no longer R16.1, R17.1, R18.1
- net G_LED: now also R17.2
- net R_LED: now also R16.2
- new net: J5.2 (Pin_2), R18.1
- new net: J5.3 (Pin_3), R17.1
- new net: J5.4 (Pin_4), R16.1
Other:
- moved on the sheet: J1, R16, R17, R18

Commit message: Last push befor ordering
Parts:
- SW1: footprint Button_Switch_SMD:SW_DIP_SPSTx01_Slide_Copal_CVS-01xB_W5.9mm_P1mm -> Button_Switch_SMD:SW_SPST_B3U-1000P
Changed lines of the file:
@@
 F 0 "SW1" H 3150 3085 50  0000 C CNN
 F 1 "SW_DPST_x2" H 3150 2994 50  0000 C CNN
-F 2 "Button_Switch_SMD:SW_DIP_SPSTx01_Slide_Copal_CVS-01xB_W5.9mm_P1mm" H 3150 2850 50  0001 C CNN
+F 2 "Button_Switch_SMD:SW_SPST_B3U-1000P" H 3150 2850 50  0001 C CNN
 F 3 "~" H 3150 2850 50  0001 C CNN
 	1    3150 2850

Commit message: added pers things to project
Parts:
- C2, C3: value 22uF -> 22pF
Changed lines of the file:
@@
 AR Path="/6022F0F9/602BBD1B" Ref="C2"  Part="1"
 F 0 "C2" V 3400 3750 50  0000 C CNN
-F 1 "22uF" V 3500 3750 50  0000 C CNN
+F 1 "22pF" V 3500 3750 50  0000 C CNN
 F 2 "Capacitor_SMD:C_0805_2012Metric_Pad1.18x1.45mm_HandSolder" H 3688 3600 50  0001 C CNN
 F 3 "~" H 3650 3750 50  0001 C CNN
@@
 AR Path="/6022F0F9/602BEADA" Ref="C3"  Part="1"
 F 0 "C3" V 3800 4150 50  0000 C CNN
-F 1 "22uF" V 3900 4150 50  0000 C CNN
+F 1 "22pF" V 3900 4150 50  0000 C CNN
 F 2 "Capacitor_SMD:C_0805_2012Metric_Pad1.18x1.45mm_HandSolder" H 3688 4000 50  0001 C CNN
 F 3 "~" H 3650 4150 50  0001 C CNN
